File: pcb/hd-mcu-v2/hd-mcu-v2.kicad_pcb (KiCad board)
At the start: 2 copper layers, 70 x 48 mm, 30 parts

Commit message: Serial commands (#5)
* add serial commands

* fix peripheral alloc

* serialize json & stream at once per service

* switch to index based keys

* remote tsm

* update pcb

* update bt serial

* fix serial com sw
Parts:
- 2: moved to B.Cu
- turned 2 to 0 degrees
Changed lines of the file:
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@@
-    )
-  )
-  (footprint "Connector_PinHeader_2.54mm:Socker_PinHeader_1x05_P2.54mm_Dualside" (layer "F.Cu")
-    (at 85.2025 75.1875 180)
-    (descr "Through hole straight pin header, 1x05, 2.54mm pitch, single row")
-    (tags "Through hole pin header THT 1x05 2.54mm single row")
-    (attr through_hole)
-    (fp_text reference "2" (at -0.44 12.54 90) (layer "B.SilkS")
-        (effects (font (size 1 1) (thickness 0.1)) (justify mirror))
-    )
-    (fp_text value "N4" (at 0 12.49) (layer "F.Fab") hide
-        (effects (font (size 1 1) (thickness 0.1)))
-    )
-    (fp_line (start 2.5 -1.8) (end 2.5 11.95)
-      (stroke (width 0.1) (type default)) (layer "B.SilkS"))
-    (fp_rect (start -1.8 -1.8) (end 3.2 11.95)
-      (stroke (width 0.1) (type default)) (fill none) (layer "B.SilkS"))
-    (fp_line (start -1.33 -1.33) (end 0 -1.33)
-      (stroke (width 0.12) (type solid)) (layer "F.SilkS"))
-    (fp_line (start -1.33 0) (end -1.33 -1.33)
-      (stroke (width 0.12) (type solid)) (layer "F.SilkS"))
-    (fp_line (start -1.33 1.27) (end -1.33 11.49)
-      (stroke (width 0.12) (type solid)) (layer "F.SilkS"))
-    (fp_line (start -1.33 1.27) (end 1.33 1.27)
-      (stroke (width 0.12) (type solid)) (layer "F.SilkS"))
-    (fp_line (start -1.33 11.49) (end 1.33 11.49)
-      (stroke (width 0.12) (type solid)) (layer "F.SilkS"))
-    (fp_line (start 1.33 1.27) (end 1.33 11.49)
-      (stroke (width 0.12) (type solid)) (layer "F.SilkS"))
-    (fp_line (start 2.5 -1.8) (end 2.5 11.95)
-      (stroke (width 0.1) (type default)) (layer "F.SilkS"))
-    (fp_rect (start -1.8 11.95) (end 3.2 -1.8)
-      (stroke (width 0.1) (type default)) (fill none) (layer "F.SilkS"))
-    (fp_line (start -1.8 -1.8) (end -1.8 11.95)
-      (stroke (width 0.05) (type solid)) (layer "F.CrtYd"))
-    (fp_line (start -1.8 11.95) (end 1.8 11.95)
-      (stroke (width 0.05) (type solid)) (layer "F.CrtYd"))
-    (fp_line (start 1.8 -1.8) (end -1.8 -1.8)
-      (stroke (width 0.05) (type solid)) (layer "F.CrtYd"))
-    (fp_line (start 1.8 11.95) (end 1.8 -1.8)
-      (stroke (width 0.05) (type solid)) (layer "F.CrtYd"))
-    (fp_line (start -1.27 -0.635) (end -0.635 -1.27)
-      (stroke (width 0.1) (type solid)) (layer "F.Fab"))
-    (fp_line (start -1.27 11.43) (end -1.27 -0.635)
-      (stroke (width 0.1) (type solid)) (layer "F.Fab"))
-    (fp_line (start -0.635 -1.27) (end 1.27 -1.27)
-      (stroke (width 0.1) (type solid)) (layer "F.Fab"))
-    (fp_line (start 1.27 -1.27) (end 1.27 11.43)
-      (stroke (width 0.1) (type solid)) (layer "F.Fab"))
-    (fp_line (start 1.27 11.43) (end -1.27 11.43)
-      (stroke (width 0.1) (type solid)) (layer "F.Fab"))
-    (pad "1" thru_hole circle (at 0 0 180) (size 1.7 1.7) (drill 1) (layers "*.Cu" "*.Mask")
-      (net 7 "5V"))
-    (pad "2" thru_hole rect (at 0 2.54 180) (size 1.7 1.7) (drill 1) (layers "*.Cu" "*.Mask")
-      (net 1 "GND"))
-    (pad "3" thru_hole oval (at 0 5.08 180) (size 1.7 1.7) (drill 1) (layers "*.Cu" "*.Mask")
-      (net 31 "D_SCK"))
-    (pad "4" thru_hole oval (at 0 7.62 180) (size 1.7 1.7) (drill 1) (layers "*.Cu" "*.Mask")
-      (net 32 "D_CS"))
-    (pad "5" thru_hole roundrect (at 0 10.16 180) (size 1.7 1.7) (drill 1) (layers "*.Cu" "*.Mask") (roundrect_rratio 0)
-      (chamfer_ratio 0.2) (chamfer top_left)
-      (net 17 "MUX_S2"))
-    (model "${KICAD6_3DMODEL_DIR}/Connector_PinHeader_2.54mm.3dshapes/PinHeader_1x05_P2.54mm_Vertical.wrl"
-      (offset (xyz 0 0 0))
-      (scale (xyz 1 1 1))
-      (rotate (xyz 0 0 0))
     )
   )
@@
       (offset (xyz 0 0 0))
       (scale (xyz 1 1 1))
+      (rotate (xyz 0 0 0))
+    )
+  )
+  (footprint "Connector_PinHeader_2.54mm:Socker_PinHeader_1x05_P2.54mm_Dualside" (layer "B.Cu")
+    (at 85.2025 75.1875)
+    (descr "Through hole straight pin header, 1x05, 2.54mm pitch, single row")
+    (tags "Through hole pin header THT 1x05 2.54mm single row")
+    (attr through_hole)
+    (fp_text reference "2" (at -0.44 -12.54 90) (layer "F.SilkS")
+        (effects (font (size 1 1) (thickness 0.1)))
+    )
+    (fp_text value "N4" (at 0 -12.49 -360) (layer "B.Fab") hide
+        (effects (font (size 1 1) (thickness 0.1)) (justify mirror))
+    )
+    (fp_line (start -1.33 -11.49) (end 1.33 -11.49)
+      (stroke (width 0.12) (type solid)) (layer "B.SilkS"))
+    (fp_line (start -1.33 -1.27) (end -1.33 -11.49)
+      (stroke (width 0.12) (type solid)) (layer "B.SilkS"))
+    (fp_line (start -1.33 -1.27) (end 1.33 -1.27)
+      (stroke (width 0.12) (type solid)) (layer "B.SilkS"))
+    (fp_line (start -1.33 0) (end -1.33 1.33)
+      (stroke (width 0.12) (type solid)) (layer "B.SilkS"))
+    (fp_line (start -1.33 1.33) (end 0 1.33)
+      (stroke (width 0.12) (type solid)) (layer "B.SilkS"))
+    (fp_line (start 1.33 -1.27) (end 1.33 -11.49)
+      (stroke (width 0.12) (type solid)) (layer "B.SilkS"))
+    (fp_line (start 2.5 1.8) (end 2.5 -11.95)
+      (stroke (width 0.1) (type default)) (layer "B.SilkS"))
+    (fp_rect (start -1.8 -11.95) (end 3.2 1.8)
+      (stroke (width 0.1) (type default)) (fill none) (layer "B.SilkS"))
+    (fp_line (start 2.5 1.8) (end 2.5 -11.95)
+      (stroke (width 0.1) (type default)) (layer "F.SilkS"))
+    (fp_rect (start -1.8 1.8) (end 3.2 -11.95)
+      (stroke (width 0.1) (type default)) (fill none) (layer "F.SilkS"))
+    (fp_line (start -1.8 -11.95) (end 1.8 -11.95)
+      (stroke (width 0.05) (type solid)) (layer "B.CrtYd"))
+    (fp_line (start -1.8 1.8) (end -1.8 -11.95)
+      (stroke (width 0.05) (type solid)) (layer "B.CrtYd"))
+    (fp_line (start 1.8 -11.95) (end 1.8 1.8)
+      (stroke (width 0.05) (type solid)) (layer "B.CrtYd"))
+    (fp_line (start 1.8 1.8) (end -1.8 1.8)
+      (stroke (width 0.05) (type solid)) (layer "B.CrtYd"))
+    (fp_line (start -1.27 -11.43) (end -1.27 0.635)
+      (stroke (width 0.1) (type solid)) (layer "B.Fab"))
+    (fp_line (start -1.27 0.635) (end -0.635 1.27)
+      (stroke (width 0.1) (type solid)) (layer "B.Fab"))
+    (fp_line (start -0.635 1.27) (end 1.27 1.27)
+      (stroke (width 0.1) (type solid)) (layer "B.Fab"))
+    (fp_line (start 1.27 -11.43) (end -1.27 -11.43)
+      (stroke (width 0.1) (type solid)) (layer "B.Fab"))
+    (fp_line (start 1.27 1.27) (end 1.27 -11.43)
+      (stroke (width 0.1) (type solid)) (layer "B.Fab"))
+    (pad "1" thru_hole circle (at 0 0) (size 1.7 1.7) (drill 1) (layers "*.Cu" "*.Mask")
+      (net 7 "5V"))
+    (pad "2" thru_hole rect (at 0 -2.54) (size 1.7 1.7) (drill 1) (layers "*.Cu" "*.Mask")
+      (net 1 "GND"))
+    (pad "3" thru_hole oval (at 0 -5.08) (size 1.7 1.7) (drill 1) (layers "*.Cu" "*.Mask")
+      (net 31 "D_SCK"))
+    (pad "4" thru_hole oval (at 0 -7.62) (size 1.7 1.7) (drill 1) (layers "*.Cu" "*.Mask")
+      (net 32 "D_CS"))
+    (pad "5" thru_hole roundrect (at 0 -10.16) (size 1.7 1.7) (drill 1) (layers "*.Cu" "*.Mask") (roundrect_rratio 0)
+      (chamfer_ratio 0.2) (chamfer bottom_left)
+      (net 17 "MUX_S2"))
+    (model "${KICAD6_3DMODEL_DIR}/Connector_PinHeader_2.54mm.3dshapes/PinHeader_1x05_P2.54mm_Vertical.wrl"
+      (offset (xyz 0 0 0))
+      (scale (xyz 1 1 1))

Commit message: wip pcb
Parts:
- added REF**: RPi_Pico_SMD_TH, denolk:RPi_Pico_SMD_TH, F.Cu at (68.4, 122.0)
Other:
- board size 70 x 48 mm -> 70 x 116.4 mm
